Commit message: Added color definitions in robot-core

File: description/robot_core.xacro (robot description, xacro)
@@ -1,4 +1,15 @@
 <?xml version="1.0"?>
 <robot xmlns:xacro="http://www.ros.org/wiki/xacro">
-    ... all our links and joints will go in here ...
+    <material name="white">
+    <color rgba="1 1 1 1"/>
+    </material>
+    <material name="orange">
+    <color rgba="1 0.3 0.1 1"/>
+    </material>
+    <material name="blue">
+    <color rgba="0.2 0.2 1 1"/>
+    </material>
+    <material name="black">
+    <color rgba="0 0 0 1"/>
+    </material>
 </robot>

Commit message: Added base link

File: description/robot_core.xacro (robot description, xacro)
@@ -13,3 +13,5 @@
     <color rgba="0 0 0 1"/>
     </material>
+    <link name="base_link">
+    </link>
 </robot>

Commit message: added the chassis link and joints

File: description/robot_core.xacro (robot description, xacro)
@@ -2,16 +2,30 @@
 <robot xmlns:xacro="http://www.ros.org/wiki/xacro">
     <material name="white">
-    <color rgba="1 1 1 1"/>
+        <color rgba="1 1 1 1"/>
     </material>
     <material name="orange">
-    <color rgba="1 0.3 0.1 1"/>
+        <color rgba="1 0.3 0.1 1"/>
     </material>
     <material name="blue">
-    <color rgba="0.2 0.2 1 1"/>
+        <color rgba="0.2 0.2 1 1"/>
     </material>
     <material name="black">
-    <color rgba="0 0 0 1"/>
+        <color rgba="0 0 0 1"/>
     </material>
     <link name="base_link">
     </link>
+    <joint name="chassis_joint" type="fixed">
+        <parent link="base_link"/>
+        <child link="chassis"/>
+        <origin xyz="-0.1 0 0"/>
+    </joint>
+    <link name="chassis">
+        <visual>
+            <origin xyz="0.15 0 0.075" rpy="0 0 0"/>
+            <geometry>
+                <box size="0.3 0.3 0.15"/>
+            </geometry>
+            <material name="white"/>
+        </visual>
+    </link>
 </robot>

Commit message: Added caster wheel links and joints

File: description/robot_core.xacro (robot description, xacro)
@@ -30,3 +30,47 @@
         </visual>
     </link>
+    <!-- LEFT WHEEL -->
+    <joint name="left_wheel_joint" type="continuous">
+        <parent link="base_link"/>
+        <child link="left_wheel"/>
+        <origin xyz="0 0.175 0" rpy="-${pi/2} 0 0"/>
+        <axis xyz="0 0 1"/>
+    </joint>
+    <link name="left_wheel">
+        <visual>
+            <geometry>
+                <cylinder length="0.04" radius="0.05" />
+            </geometry>
+            <material name="blue"/>
+        </visual>
+    </link>
+    <!-- RIGHT WHEEL -->
+    <joint name="right_wheel_joint" type="continuous">
+        <parent link="base_link"/>
+        <child link="right_wheel"/>
+        <origin xyz="0 -0.175 0" rpy="${pi/2} 0 0"/>
+        <axis xyz="0 0 -1"/>
+    </joint>
+    <link name="right_wheel">
+        <visual>
+            <geometry>
+                <cylinder length="0.04" radius="0.05" />
+            </geometry>
+            <material name="blue"/>
+        </visual>
+    </link>
+    <!-- CASTER WHEEL -->
+    <joint name="caster_wheel_joint" type="fixed">
+        <parent link="chassis"/>
+        <child link="caster_wheel"/>
+        <origin xyz="0.24 0 0" rpy="0 0 0"/>
+    </joint>
+    <link name="caster_wheel">
+        <visual>
+            <geometry>
+                <sphere radius="0.05" />
+            </geometry>
+            <material name="black"/>
+        </visual>
+    </link>
 </robot>

Commit message: Add the collision tags for chassis and the wheels

File: description/robot_core.xacro (robot description, xacro)
@@ -29,4 +29,10 @@
             <material name="white"/>
         </visual>
+        <collision>
+            <origin xyz="0.15 0 0.075" rpy="0 0 0"/>
+            <geometry>
+                <box size="0.3 0.3 0.15"/>
+            </geometry>
+        </collision>
     </link>
     <!-- LEFT WHEEL -->
@@ -44,4 +50,9 @@
             <material name="blue"/>
         </visual>
+        <collision>
+            <geometry>
+                <cylinder length="0.04" radius="0.05" />
+            </geometry>
+        </collision>
     </link>
     <!-- RIGHT WHEEL -->
@@ -59,4 +70,9 @@
             <material name="blue"/>
         </visual>
+        <collision>
+            <geometry>
+                <cylinder length="0.04" radius="0.05" />
+            </geometry>
+        </collision>
     </link>
     <!-- CASTER WHEEL -->
@@ -73,4 +89,9 @@
             <material name="black"/>
         </visual>
+        <collision>
+            <geometry>
+                <sphere radius="0.05" />
+            </geometry>
+        </collision>
     </link>
 </robot>

Commit message: Added inertia tags to chassis and wheels

File: description/robot_core.xacro (robot description, xacro)
@@ -36,4 +36,7 @@
             </geometry>
         </collision>
+        <xacro:inertial_box mass="0.5" x="0.3" y="0.3" z="0.15">
+        <origin xyz="0.15 0 0.075" rpy="0 0 0"/>
+    </xacro:inertial_box>
     </link>
     <!-- LEFT WHEEL -->
@@ -56,4 +59,7 @@
             </geometry>
         </collision>
+        <xacro:inertial_cylinder mass="0.1" length="0.05" radius="0.05">
+        <origin xyz="0 0 0" rpy="0 0 0"/>
+        </xacro:inertial_cylinder>
     </link>
     <!-- RIGHT WHEEL -->
@@ -76,4 +82,8 @@
             </geometry>
         </collision>
+        <!-- Same as left wheel-->
+        <xacro:inertial_cylinder mass="0.1" length="0.05" radius="0.05">
+        <origin xyz="0 0 0" rpy="0 0 0"/>
+        </xacro:inertial_cylinder>
     </link>
     <!-- CASTER WHEEL -->
@@ -95,4 +105,7 @@
             </geometry>
         </collision>
+         <xacro:inertial_sphere mass="0.1" radius="0.05">
+        <origin xyz="0 0 0" rpy="0 0 0"/>
+    </xacro:inertial_sphere>
     </link>
 </robot>

Commit message: added gazebo tags with material color for chassis and wheels

File: description/robot_core.xacro (robot description, xacro)
@@ -40,4 +40,7 @@
     </xacro:inertial_box>
     </link>
+    <gazebo reference="chassis">
+        <material>Gazebo/White</material>
+    </gazebo>
     <!-- LEFT WHEEL -->
     <joint name="left_wheel_joint" type="continuous">
@@ -63,4 +66,7 @@
         </xacro:inertial_cylinder>
     </link>
+    <gazebo reference="left_wheel">
+        <material>Gazebo/Blue</material>
+    </gazebo>
     <!-- RIGHT WHEEL -->
     <joint name="right_wheel_joint" type="continuous">
@@ -87,4 +93,7 @@
         </xacro:inertial_cylinder>
     </link>
+    <gazebo reference="right_wheel">
+        <material>Gazebo/Blue</material>
+    </gazebo>
     <!-- CASTER WHEEL -->
     <joint name="caster_wheel_joint" type="fixed">
@@ -109,3 +118,6 @@
     </xacro:inertial_sphere>
     </link>
+    <gazebo reference="caster_wheel">
+        <material>Gazebo/Black</material>
+    </gazebo>
 </robot>
