Commit message: emergency commit

File: description/robot.urdf.xacro (robot description, xacro)
@@ -1,5 +1,22 @@
 <?xml version="1.0"?>
 <robot xmlns:xacro="http://www.ros.org/wiki/xacro"  name="robot">
-    1<xacro:include filename="robot_core.xacro" />
-    1<xacro:include filename="gazebo_control.xacro" />
+    <xacro:include filename="robot_core.xacro" />
+    <xacro:include filename="gazebo_control.xacro" />
+    <xacro:include filename="ultrasonic_sensor.xacro" />
 </robot>
+    <!--  -->
+    <!-- <xacro:ultrasonic_sensor sensor_name="front_left_sensor" parent_link="chassis">
+    <origin xyz="0.25 0.15 0.15" rpy="0 0 0"/>
+    </xacro:ultrasonic_sensor> -->
+    <!-- <xacro:ultrasonic_sensor sensor_name="front_center_sensor" parent_link="chassis">
+    <origin xyz="0.30 0 0.15" rpy="0 0 0"/>
+    </xacro:ultrasonic_sensor>
+    <xacro:ultrasonic_sensor sensor_name="front_right_sensor" parent_link="chassis">
+    <origin xyz="0.25 -0.15 0.15" rpy="0 0 0"/>
+    </xacro:ultrasonic_sensor>
+    <xacro:ultrasonic_sensor sensor_name="rear_left_sensor" parent_link="chassis">
+    <origin xyz="0.05 0.15 0.15" rpy="0 0 ${pi}"/>
+    </xacro:ultrasonic_sensor>
+    <xacro:ultrasonic_sensor sensor_name="rear_right_sensor" parent_link="chassis">
+    <origin xyz="0.05 -0.15 0.15" rpy="0 0 ${pi}"/>
+    </xacro:ultrasonic_sensor> -->

File: description/robot_core.xacro (robot description, xacro)
@@ -13,4 +13,7 @@
     <material name="black">
         <color rgba="0 0 0 1"/>
+    </material>
+    <material name="red">
+        <color rgba="1 0 0 1"/>
     </material>
     <!--Base Link-->
