Commit message: last commit before migration to ROS Jazzy and Ubuntu 24.04

File: description/gazebo_control.xacro (robot description, xacro)
@@ -1,21 +1,30 @@
 <?xml version="1.0"?>
 <robot xmlns:xacro="http://www.ros.org/wiki/xacro">
-    <gazebo>
-        <plugin name='diff_drive' filename='libgazebo_ros_diff_drive.so'>
-            <!-- Wheel Information -->
-            <left_joint>left_wheel_joint</left_joint>
-            <right_joint>right_wheel_joint</right_joint>
-            <wheel_separation>0.35</wheel_separation>
-            <wheel_diameter>0.1</wheel_diameter>
-            <!-- Limits -->
-            <max_wheel_torque>200</max_wheel_torque>
-            <max_wheel_acceleration>10.0</max_wheel_acceleration>
-            <!-- Output -->
-            <odometry_frame>odom</odometry_frame>
-            <robot_base_frame>base_link</robot_base_frame>
-            <publish_odom>true</publish_odom>
-            <publish_odom_tf>true</publish_odom_tf>
-            <publish_wheel_tf>true</publish_wheel_tf>
-        </plugin>
-    </gazebo>
+  <gazebo>
+    <plugin name="diff_drive" filename="libgazebo_ros_diff_drive.so">
+      <!-- ROS 2 parameters -->
+      <ros>
+        <namespace>/</namespace>
+      </ros>
+      <!-- Wheel Information -->
+      <left_joint>left_wheel_joint</left_joint>
+      <right_joint>right_wheel_joint</right_joint>
+      <wheel_separation>0.35</wheel_separation>
+      <wheel_diameter>0.1</wheel_diameter>
+      <!-- Odometry and TF -->
+      <odometry_frame>odom</odometry_frame>
+      <robot_base_frame>base_link</robot_base_frame>
+      <publish_odom>true</publish_odom>
+      <publish_odom_tf>true</publish_odom_tf>
+      <publish_wheel_tf>false</publish_wheel_tf>
+      <!-- Output Topics -->
+      <odometry_topic>odom</odometry_topic>
+      <cmd_vel_topic>cmd_vel</cmd_vel_topic>
+      <!-- Limits -->
+      <max_wheel_torque>200</max_wheel_torque>
+      <max_wheel_acceleration>10.0</max_wheel_acceleration>
+      <!-- Simulation Parameters -->
+      <update_rate>50</update_rate>
+    </plugin>
+  </gazebo>
 </robot>

File: description/robot.urdf.xacro (robot description, xacro)
@@ -5,18 +5,2 @@
     <xacro:include filename="ultrasonic_sensor.xacro" />
 </robot>
-    <!--  -->
-    <!-- <xacro:ultrasonic_sensor sensor_name="front_left_sensor" parent_link="chassis">
-    <origin xyz="0.25 0.15 0.15" rpy="0 0 0"/>
-    </xacro:ultrasonic_sensor> -->
-    <!-- <xacro:ultrasonic_sensor sensor_name="front_center_sensor" parent_link="chassis">
-    <origin xyz="0.30 0 0.15" rpy="0 0 0"/>
-    </xacro:ultrasonic_sensor>
-    <xacro:ultrasonic_sensor sensor_name="front_right_sensor" parent_link="chassis">
-    <origin xyz="0.25 -0.15 0.15" rpy="0 0 0"/>
-    </xacro:ultrasonic_sensor>
-    <xacro:ultrasonic_sensor sensor_name="rear_left_sensor" parent_link="chassis">
-    <origin xyz="0.05 0.15 0.15" rpy="0 0 ${pi}"/>
-    </xacro:ultrasonic_sensor>
-    <xacro:ultrasonic_sensor sensor_name="rear_right_sensor" parent_link="chassis">
-    <origin xyz="0.05 -0.15 0.15" rpy="0 0 ${pi}"/>
-    </xacro:ultrasonic_sensor> -->

File: description/ultrasonic_sensor.xacro (robot description, xacro)
@@ -5,6 +5,7 @@
         <parent link="chassis"/>
         <child link="front_left_sensor_link"/>
-        <origin xyz="0.25 0.15 0.15" rpy="0 0 0"/>
-        <axis xyz="0 1 0"/> <!-- Rotate around Y-axis -->
+        <!-- <origin xyz="0.25 0.15 0.15" rpy="0 0 0"/> -->
+        <origin xyz="0.32 0.15 0.16" rpy="0 0 0"/>
+        <!-- <axis xyz="0 1 0"/> -->
     </joint>
     <!-- make the sensor like one of the wheels-->
@@ -12,5 +13,5 @@
     <visual>
             <geometry>
-                <cylinder length="0.04" radius="0.05" />
+                <cylinder length="0.02" radius="0.02"/>
             </geometry>
             <material name="red"/>
@@ -18,9 +19,9 @@
         <collision>
             <geometry>
-                <cylinder length="0.04" radius="0.05" />
+                <cylinder length="0.02" radius="0.02"/>
             </geometry>
         </collision>
-        <xacro:inertial_cylinder mass="0.1" length="0.05" radius="0.05">
-        <origin xyz="0 0 0" rpy="0 0 0"/>
+        <xacro:inertial_cylinder mass="0.1" length="0.02" radius="0.02">
+          <origin xyz="0 0 0" rpy="0 0 0"/>
         </xacro:inertial_cylinder>
     </link>
@@ -30,5 +31,5 @@
         <pose>0 0 0 0 0 0</pose> <!-- Relative pose to the sensor link -->
         <always_on>true</always_on>
-        <visualize>false</visualize>
+        <visualize>true</visualize>
         <update_rate>5</update_rate>
         <ray>
@@ -37,12 +38,12 @@
               <samples>5</samples>
               <resolution>1.000000</resolution>
-              <min_angle>-0.12</min_angle>
-              <max_angle>0.12</max_angle>
+              <min_angle>-0.131</min_angle>  <!-- -7.5 degrees -->
+              <max_angle>0.131</max_angle>   <!-- +7.5 degrees -->
             </horizontal>
             <vertical>
-              <samples>5</samples>
+              <samples>1</samples>
               <resolution>1.000000</resolution>
-              <min_angle>-0.01</min_angle>
-              <max_angle>0.01</max_angle>
+              <min_angle>0.0</min_angle>
+              <max_angle>0.0</max_angle>
             </vertical>
           </scan>
@@ -59,12 +60,11 @@
         </ray>
         <plugin name="ultrasonic_front_left" filename="libgazebo_ros_ray_sensor.so">
-          <ros>
-            <namespace>/</namespace> <!-- publish to global namespace -->
-          </ros>
-          <topic_name>ultrasonic_front_left</topic_name>
-          <output_type>sensor_msgs/Range</output_type>
-          <radiation_type>ultrasound</radiation_type>
-          <frame_name>front_left_sensor_link</frame_name>
-      </plugin>
+            <ros>
+              <remapping>~/out:=/ultrasonic_front_left</remapping>
+            </ros>
+            <output_type>sensor_msgs/Range</output_type>
+            <radiation_type>ultrasound</radiation_type>
+            <frame_name>front_left_sensor_link</frame_name>
+        </plugin>
       </sensor>
   </gazebo>
